File: Franzininho - PCB/PCB_CNC/Franzininho_CNC.brd (EAGLE design)
At the start: 53.1 x 26.1 mm, 16 parts, among them IC1 TINY45-20-DIP, X1 USBPCB

Commit message: atualização de arquivos
Parts:
- IC1: value TINY45-20-DIP -> ATTINY85 - 20PU
Changed lines of the file:
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@@
 <attribute name="VALUE" x="2.62" y="17.17" size="0.4064" layer="28" rot="MR180"/>
 </element>
-<element name="IC1" library="SparkFun-DigitalIC" package="DIP08" value="TINY45-20-DIP" x="39.2316" y="12.0435" smashed="yes" rot="R180">
+<element name="IC1" library="SparkFun-DigitalIC" package="DIP08" value="ATTINY85 - 20PU" x="39.2316" y="12.0435" smashed="yes" rot="R180">
 <attribute name="PROD_ID" value="IC-09439" x="39.2316" y="12.0435" size="1.778" layer="27" rot="R180" display="off"/>
 <attribute name="VALUE" value="TINY45-20-DIP" x="39.2316" y="12.0435" size="1.778" layer="27" rot="R180" display="off"/>
