File: Franzininho - PCB/PCB_CNC/Franzininho_CNC.sch (EAGLE design)
At the start: 16 parts, among them IC1 TINY45-20-DIP, X1 USBPCB

Commit message: atualização de arquivos
Parts:
- IC1: value TINY45-20-DIP -> ATTINY85 - 20PU
Changed lines of the file:
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@@
 <parts>
 <part name="X1" library="SparkFun" deviceset="USB" device="PCB"/>
-<part name="IC1" library="SparkFun-DigitalIC" deviceset="ATTINY45" device="TINY45-20-DIP" value="TINY45-20-DIP"/>
+<part name="IC1" library="SparkFun-DigitalIC" deviceset="ATTINY45" device="TINY45-20-DIP" value="ATTINY85 - 20PU"/>
 <part name="D2" library="SparkFun-DiscreteSemi" deviceset="DIODE-ZENER" device="" value="BZT52"/>
 <part name="D1" library="SparkFun-DiscreteSemi" deviceset="DIODE-ZENER" device="" value="BZT52"/>
