File: hardware/Franzininho - V2 - Eagle/Franzininho.brd (EAGLE design)
At the start: 51.1 x 30 mm, 19 parts, among them IC1 ATTINY85 - 20PU, X1 USB-A-H

Commit message: correção do conector USB
Parts:
- moved X1 0.17 mm to (13.9, 16.2), flipped to the top, turned to 0 degrees
Routing:
- net N$4: track 6.59 -> 32.4 mm
- net GND: track 24.8 -> 0.00 mm
- net N$10: track 19.3 -> 26.6 mm
- net N$11: track 7.47 -> 8.21 mm
Other:
- board text added: "Acesse: www.franzininho.com.br"
- board text removed: "Acesse: www.embarcados.com.br/franzininho"
