File: Franzininho - RV1/Franzininho - RV1 - KiCAD/franzininho-rev1.sch (KiCad schematic (older format))
At the start: 17 parts, among them J1 CONN_01X08, SW1 SW_RESET, U1 ATTINY85-20PU, U2 USB_conn

Commit message: Compatibilidade Multiplataforma (Kicad Rev1) - Issue #21
Parts:
- C1: symbol C -> Device:C
- C2: symbol CP1 -> Device:CP1
- D1, D2: symbol D_Zener -> Device:D_Zener
- D3: symbol D -> Device:D
- D4, D5: symbol LED -> Device:LED
- J1: symbol CONN_01X08 -> franzininho-rev1:CONN_01X08
- LOGO1: symbol OPEN_HARDWARE_1 -> franzininho-rev1:OPEN_HARDWARE_1
- R1, R2, R3, R4, R5: symbol R -> Device:R
- SW1: symbol SW_Push -> franzininho-rev1:SW_Push
- U1: symbol ATTINY85-20PU -> franzininho-rev1:ATTINY85-20PU
- U2: symbol USB_conn -> franzininho-rev1:USB_conn
Changed lines of the file:
@@
-EESchema Schematic File Version 2
-LIBS:power
-LIBS:device
-LIBS:transistors
-LIBS:conn
-LIBS:linear
-LIBS:regul
-LIBS:74xx
-LIBS:cmos4000
-LIBS:adc-dac
-LIBS:memory
-LIBS:xilinx
-LIBS:microcontrollers
-LIBS:dsp
-LIBS:microchip
-LIBS:analog_switches
-LIBS:motorola
-LIBS:texas
-LIBS:intel
-LIBS:audio
-LIBS:interface
-LIBS:digital-audio
-LIBS:philips
-LIBS:display
-LIBS:cypress
-LIBS:siliconi
-LIBS:opto
-LIBS:atmel
-LIBS:contrib
-LIBS:valves
-LIBS:usb_conn
-LIBS:ttl_ieee
-LIBS:sensors
-LIBS:switches
-LIBS:supertex
-LIBS:powerint
-LIBS:wiznet
-LIBS:onsemi
-LIBS:stm32
-LIBS:nordicsemi
-LIBS:transf
-LIBS:references
-LIBS:rfcom
-LIBS:relays
-LIBS:silabs
-LIBS:triac_thyristor
-LIBS:nxp
-LIBS:zetex
-LIBS:pspice
-LIBS:nxp_armmcu
-LIBS:video
-LIBS:msp430
-LIBS:stm8
-LIBS:ir
-LIBS:Oscillators
-LIBS:bbd
-LIBS:gennum
-LIBS:modules
-LIBS:microchip_pic24mcu
-LIBS:motor_drivers
-LIBS:microchip_dspic33dsc
-LIBS:dc-dc
-LIBS:ESD_Protection
-LIBS:elec-unifil
-LIBS:diode
-LIBS:graphic
-LIBS:microchip_pic18mcu
-LIBS:maxim
-LIBS:microchip_pic32mcu
-LIBS:Zilog
-LIBS:Lattice
-LIBS:hc11
-LIBS:Altera
-LIBS:actel
-LIBS:Worldsemi
-LIBS:cmos_ieee
-LIBS:microchip_pic16mcu
-LIBS:logo
-LIBS:motors
-LIBS:microchip_pic12mcu
-LIBS:analog_devices
-LIBS:Xicor
-LIBS:Power_Management
-LIBS:74xgxx
-LIBS:ftdi
-LIBS:mechanical
-LIBS:brooktre
-LIBS:allegro
-LIBS:battery_management
-LIBS:microchip_pic10mcu
-LIBS:bosch
-LIBS:leds
-LIBS:ac-dc
+EESchema Schematic File Version 4
 LIBS:franzininho-rev1-cache
-EELAYER 25 0
+EELAYER 26 0
 EELAYER END
 $Descr A4 11693 8268
@@
 $EndDescr
 $Comp
-L USB_conn U2
+L franzininho-rev1:USB_conn U2
 U 1 1 595ECB99
 P 3250 3925
@@
 $EndComp
 $Comp
-L ATTINY85-20PU U1
+L franzininho-rev1:ATTINY85-20PU U1
 U 1 1 595ECBDF
 P 6025 3625
@@
 $EndComp
 $Comp
-L PWR_FLAG #FLG01
+L power:PWR_FLAG #FLG01
 U 1 1 595ECD5A
 P 3450 2700
@@
 $EndComp
 $Comp
-L PWR_FLAG #FLG02
+L power:PWR_FLAG #FLG02
 U 1 1 595ECD72
 P 3800 2575
@@
 $EndComp
 $Comp
-L +5V #PWR03
+L power:+5V #PWR03
 U 1 1 595ECD8A
 P 3625 3300
@@
 $EndComp
 $Comp
-L GND #PWR04
+L power:GND #PWR04
 U 1 1 595ECDA2
 P 3650 4200
@@
 $EndComp
 $Comp
-L CP1 C2
+L Device:CP1 C2
 U 1 1 595ECE64
 P 2600 3125
@@
 $EndComp
 $Comp
-L R R1
+L Device:R R1
 U 1 1 595ECE9C
 P 4625 4350
@@
 $EndComp
 $Comp
-L R R2
+L Device:R R2
 U 1 1 595ECEFD
 P 4625 4575
@@
 $EndComp
 $Comp
-L R R4
+L Device:R R4
 U 1 1 595ECF43
 P 2775 4700
@@
 $EndComp
 $Comp
-L R R3
+L Device:R R3
 U 1 1 595ECF76
 P 4150 3575
@@
 $EndComp
 $Comp
-L R R5
+L Device:R R5
 U 1 1 595ECFAC
 P 8700 3475
@@
 $EndComp
 $Comp
-L LED D4
+L Device:LED D4
 U 1 1 595ECFE0
 P 2775 4225
@@
 $EndComp
 $Comp
-L LED D5
+L Device:LED D5
 U 1 1 595ED02B
 P 8275 3475
@@
 $EndComp
 $Comp
-L D D3
+L Device:D D3
 U 1 1 595ED077
 P 3625 3500
@@
 $EndComp
 $Comp
-L D_Zener D1
+L Device:D_Zener D1
 U 1 1 595ED0E8
 P 4150 4825
@@
 $EndComp
 $Comp
-L D_Zener D2
+L Device:D_Zener D2
 U 1 1 595ED13A
 P 3875 4825
@@
 $EndComp
 $Comp
-L CONN_01X08 J1
+L franzininho-rev1:CONN_01X08 J1
 U 1 1 595ED184
 P 7825 2700
@@
 $EndComp
 $Comp
-L OPEN_HARDWARE_1 LOGO1
+L franzininho-rev1:OPEN_HARDWARE_1 LOGO1
 U 1 1 595ED39D
 P 5850 2700
@@
 $EndComp
 $Comp
-L +5V #PWR05
+L power:+5V #PWR05
 U 1 1 595EE83A
 P 2775 3900
@@
 $EndComp
 $Comp
-L +5V #PWR06
+L power:+5V #PWR06
 U 1 1 595EE9C5
 P 3450 2575
@@
 $EndComp
 $Comp
-L GND #PWR07
+L power:GND #PWR07
 U 1 1 595EF3FC
 P 2775 5025
@@
 $EndComp
 $Comp
-L GND #PWR08
+L power:GND #PWR08
 U 1 1 595EFBE0
 P 4600 3950
@@
 $EndComp
 $Comp
-L +5V #PWR09
+L power:+5V #PWR09
 U 1 1 595EFC1B
 P 4600 3325
@@
 $EndComp
 $Comp
-L GND #PWR010
+L power:GND #PWR010
 U 1 1 595F11B3
 P 8975 3475
@@
 $EndComp
 $Comp
-L GND #PWR011
+L power:GND #PWR011
 U 1 1 595F2C36
 P 4000 5175
@@
 $EndComp
 $Comp
-L GND #PWR012
+L power:GND #PWR012
 U 1 1 595F3866
 P 3800 2700
@@
 $EndComp
 $Comp
-L +5V #PWR013
+L power:+5V #PWR013
 U 1 1 595F3D31
 P 2750 2800
@@
 $EndComp
 $Comp
-L GND #PWR014
+L power:GND #PWR014
 U 1 1 595F416C
 P 2775 3400
@@
 	3550 3850 4150 3850
 Wire Wire Line
-	4150 3725 4150 4675
+	4150 3725 4150 3850
 Wire Wire Line
 	3550 4000 3875 4000
@@
 	3875 4975 3875 5175
 Wire Wire Line
-	3875 5175 4150 5175
+	3875 5175 4000 5175
 Wire Wire Line
 	4150 5175 4150 4975
@@
 	2600 2975 2600 2800
 Wire Wire Line
-	2600 2800 2900 2800
+	2600 2800 2750 2800
 Connection ~ 2750 2800
 Wire Wire Line
 	2600 3275 2600 3400
 Wire Wire Line
-	2600 3400 2900 3400
+	2600 3400 2775 3400
 Connection ~ 2775 3400
 Wire Wire Line
@@
 Connection ~ 3875 4575
 $Comp
-L +5V #PWR015
+L power:+5V #PWR015
 U 1 1 595F58C7
 P 4150 3350
@@
 	7575 2900 7575 3475
 Wire Wire Line
-	7375 3475 8125 3475
+	7375 3475 7575 3475
 Wire Wire Line
 	7675 2900 7675 3575
@@
 	7775 2900 7775 3675
 Wire Wire Line
-	7775 3675 7375 3675
+	7775 3675 7475 3675
 Wire Wire Line
 	7975 2900 7975 3775
 Wire Wire Line
-	7975 3775 7375 3775
+	7975 3775 7575 3775
 Wire Wire Line
 	7875 3875 7375 3875
 $Comp
-L +5V #PWR016
+L power:+5V #PWR016
 U 1 1 595F63D6
 P 8075 3000
@@
 $EndComp
 $Comp
-L GND #PWR017
+L power:GND #PWR017
 U 1 1 595F6411
 P 8250 3000
@@
 Connection ~ 7875 3875
 $Comp
-L GND #PWR018
+L power:GND #PWR018
 U 1 1 595F7DAE
 P 7875 4825
@@
 $EndComp
 Wire Wire Line
-	3875 4000 3875 4675
-$Comp
-L C C1
+	3875 4000 3875 4575
+$Comp
+L Device:C C1
 U 1 1 595FED9B
 P 2900 3125
@@
 	2900 3400 2900 3275
 $Comp
-L SW_Push SW1
+L franzininho-rev1:SW_Push SW1
 U 1 1 595EEE76
 P 7875 4400
@@
 $EndComp
 Wire Wire Line
-	7875 2900 7875 4200
+	7875 2900 7875 3875
 Wire Wire Line
 	7875 4600 7875 4825
+Wire Wire Line
+	4000 5175 4150 5175
+Wire Wire Line
+	2750 2800 2900 2800
+Wire Wire Line
+	2775 3400 2900 3400
+Wire Wire Line
+	4150 4350 4150 4675
+Wire Wire Line
+	3875 4575 3875 4675
+Wire Wire Line
+	4150 3850 4150 4350
+Wire Wire Line
+	7575 3475 8125 3475
+Wire Wire Line
+	7475 3675 7375 3675
+Wire Wire Line
+	7575 3775 7375 3775
+Wire Wire Line
+	7875 3875 7875 4200
 $EndSCHEMATC
