File: Franzininho DIY/Franzininho.sch (KiCad schematic (older format))
At the start: 19 parts, among them IC1 ATTINY85 - 20PU, J1 M03PTH, U1 L78L05_TO92, X1 USB-A-H

Commit message: Ajustando lib 3D e gerando arquivo step
Parts:
- removed LOGO1: OSHW-LOGOM, Franzininho:OSHW-LOGO-M, symbol Franzininho-eagle-import:OSHW-LOGOM
Other:
- note removed: "FRANZININHO V2"
- note removed: "by Fábio Souza"
Changed lines of the file:
@@
 EESchema Schematic File Version 4
-LIBS:Franzininho-cache
 EELAYER 30 0
 EELAYER END
-$Descr User 11774 8268
+$Descr A4 11693 8268
 encoding utf-8
 Sheet 1 1
 Title ""
-Date ""
+Date "2021-02-06"
 Rev ""
 Comp ""
@@
 $EndComp
 $Comp
-L Franzininho-eagle-import:OSHW-LOGOM LOGO1
-U 1 1 23D986A4
-P 9500 4900
-F 0 "LOGO1" H 9500 4900 50  0001 C CNN
-F 1 "OSHW-LOGOM" H 9500 4900 50  0001 C CNN
-F 2 "Franzininho:OSHW-LOGO-M" H 9500 4900 50  0001 C CNN
-F 3 "" H 9500 4900 50  0001 C CNN
-	1    9500 4900
-	1    0    0    -1
-$EndComp
-$Comp
 L Franzininho-eagle-import:TACTILE-SWITCH-PTH RESET1
 U 1 1 1E829C81
@@
 $EndComp
 $Comp
-L Franzininho-eagle-import:A4L-LOC #FRAME1
-U 1 1 CC96BE83
-P 900 7200
-F 0 "#FRAME1" H 900 7200 50  0001 C CNN
-F 1 "A4L-LOC" H 900 7200 50  0001 C CNN
-F 2 "" H 900 7200 50  0001 C CNN
-F 3 "" H 900 7200 50  0001 C CNN
-	1    900  7200
-	1    0    0    -1
-$EndComp
-Text Notes 7400 6700 0    127  ~ 0
-FRANZININHO V2
-Text Notes 9500 6400 0    73   ~ 0
-by Fábio Souza
-$Comp
 L Regulator_Linear:L78L05_TO92 U1
